Commit message: UODATDED

File: trash/robot.urdf (robot description, URDF)
Before this commit: robot dasautonomeauto, 3 links, 2 joints
Links:
- removed link imu_link
- added link velodyne, mass 0.01; visual mesh filename=file://$(find velodyne_description)/meshes/VLP16_scan.dae
- added link velodyne_base_link, mass 0.83; collision cylinder length=0.0717 radius=0.0516; visual mesh filename=file://$(find velodyne_description)/meshes/VLP16_base_1.dae
Joints:
- removed joint imu_joint
- added joint velodyne_base_mount_joint: type fixed, parent base_link, child velodyne_base_link, origin xyz=0 0 1.8 rpy=0 3.141592653589793 0
- added joint velodyne_base_scan_joint: type fixed, parent velodyne_base_link, child velodyne, origin xyz=0 0 0.0377 rpy=0 0 0
