Commit message: updated pkgs

File: sdv_description/urdf/robot.urdf (robot description, URDF)
Before this commit: robot dasautonomeauto, 3 links, 2 joints
Links:
- link base_link: mass 10 -> 125.0

File: sdv_description/urdf/wheels_sdv.xacro (robot description, xacro)
@@ -1,6 +1,10 @@
 <?xml version="1.0"?>
 <robot name="sdv_car" xmlns:xacro="http://www.ros.org/wiki/xacro">
+<!--
+  <xacro:property name="tire_dia" value="0.750"/>
+  <xacro:property name="tire_width" value="0.125"/>
+  <xacro:property name="hub_dia" value="0.235"/>   -->
   <xacro:property name="tire_dia" value="0.750"/>  <!-- Reduced from 0.440 -->
-  <xacro:property name="tire_width" value="0.125"/>  <!-- Reduced from 0.195 -->
+  <xacro:property name="tire_width" value="0.195"/>  <!-- Reduced from 0.195 -->
   <xacro:property name="hub_dia" value="0.235"/>  <!-- Reduced from 0.235 -->
   <xacro:property name="hex_hub_depth" value="0.120"/> <!-- or +0.072 -->
@@ -43,11 +47,16 @@
   <xacro:macro name="null_inertial">
     <inertial>
-      <!-- <origin xyz="0 0 -0.02"/> -->
       <mass value="4.5"/>
-      <inertia ixx="0.00001" ixy="0" ixz="0" iyy="0.00001" iyz="0" izz="0.000004"/>
+      <inertia ixx="0.001" ixy="0" ixz="0" iyy="0.001" iyz="0" izz="0.001"/>
     </inertial>
   </xacro:macro>
   <!-- front wheel -->
   <xacro:macro name="front_wheel" params="lr_prefix fr_prefix lr_reflect">
+    <link name="${lr_prefix}_steering_link">
+      <xacro:null_inertial/>
+      <!-- <xacro:thick_walled_tube_inertial
+          inner_rad="${hub_dia / 2}" outer_rad="${tire_dia / 2}"
+          height="${tire_width}" mass="${wheel_mass}"/> -->
+    </link>
     <joint name="${lr_prefix}_steering_joint" type="revolute">
       <origin xyz="${fr_reflect * front_wheel_x} ${lr_reflect * front_wheel_y} ${-front_wheel_z}" rpy="0 ${degrees_90} 0"/>
@@ -57,24 +66,4 @@
       <limit lower="${-degrees_45}" upper="${degrees_45}"
             effort="${servo_stall_torque}" velocity="${servo_no_load_speed}"/>
-    </joint>
-    <link name="${lr_prefix}_steering_link">
-        <visual>
-            <geometry>
-                <mesh filename="file://$(find sdv_description)/meshes/DAE/suspension/front_right_sus.dae" />
-            </geometry>
-        </visual>
-        <collision>
-            <geometry>
-                <mesh filename="file://$(find sdv_description)/meshes/STL/suspension/front_right_sus.stl" />
-            </geometry>
-        </collision>
-      <xacro:null_inertial/>
-    </link>
-    <joint name="${lr_prefix}_${fr_prefix}_axle" type="continuous">
-      <parent link="${lr_prefix}_steering_link"/>
-      <child link="${lr_prefix}_${fr_prefix}_wheel"/>
-      <origin xyz="0 0 0" rpy="1.5708 0 0" />
-      <axis xyz="0 0 -1"/>
-      <limit effort="${axle_eff_limit}" velocity="${axle_vel_limit}"/>
     </joint>
     <link name="${lr_prefix}_${fr_prefix}_wheel">
@@ -100,4 +89,11 @@
           height="${tire_width}" mass="${wheel_mass}"/>
     </link>
+    <joint name="${lr_prefix}_${fr_prefix}_axle" type="continuous">
+      <parent link="${lr_prefix}_steering_link"/>
+      <child link="${lr_prefix}_${fr_prefix}_wheel"/>
+      <origin xyz="0 0 0" rpy="1.5708 0 0" />
+      <axis xyz="0 0 -1"/>
+      <limit effort="${axle_eff_limit}" velocity="${axle_vel_limit}"/>
+    </joint>
     <gazebo reference="${lr_prefix}_${fr_prefix}_wheel">
       <material>Gazebo/Black</material>
